File: hardware/TireTempSensor_v3.0/IRSensor.kicad_sch (KiCad schematic)
At the start: 7 parts, among them IC2 MLX90621ESF-BAB-000-SP

Commit message: gerber update bo wczesniej nie dzialalo; jeszcze trzeba poprawic tabele z komponentami
Parts:
- C17: footprint Capacitor_SMD:C_0603_1608Metric -> Capacitor_SMD:C_0603_1608Metric_Pad1.08x0.95mm_HandSolder; Mouser Part Number (none) -> 81-GCJ188R71H104MA2D; Mouser Price/Stock (none) -> https://www.mouser.pl/pl/ProductDetail/Murata-Electronics/G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
