File: hardware/TireTempSensor_v3.0/CAN.kicad_sch (KiCad schematic)
At the start: 21 parts, among them U7 ADM3057ExRW

Commit message: gerber update bo wczesniej nie dzialalo; jeszcze trzeba poprawic tabele z komponentami
Parts:
- C36: Mouser Part Number (none) -> 81-GCJ188R71H104MA2D; Mouser Price/Stock (none) -> https://www.mouser.pl/pl/ProductDetail/Murata-Electronics/G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
