File: hardware/TireTempSensor_v3.0/PowerSupply.kicad_sch (KiCad schematic)
At the start: 32 parts, among them IC1 TAR5S33UTE85LF, IC4 TPS54202HDDCR, T10 TP_+5V, T14 TP_+3.3V, T15 TP_+2.6V, U2 MIC5306-2.6YD5-TR

Commit message: gerber update bo wczesniej nie dzialalo; jeszcze trzeba poprawic tabele z komponentami
Parts:
- C26, C41, C42, C43: Mouser Part Number 810-C2012X5R1V226MAC -> 81-ZRA21CR61E226ME1L; Mouser Price/Stock https://www.mouser.pl/ProductDetail/TDK/C2012X5R1V226M125AC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 -> https://www.mouser.pl/pl/ProductDetail/Murata-Electronics/Z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
- C28: Mouser Part Number 80-C0603C104J3R -> 81-GCJ188R71H104MA2D; Mouser Price/Stock https://www.mouser.pl/ProductDetail/Murata-Electronics/GRM0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 -> https://www.mouser.pl/pl/ProductDetail/Murata-Electronics/G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
- C31: footprint Capacitor_SMD:C_0603_1608Metric -> Capacitor_SMD:C_0603_1608Metric_Pad1.08x0.95mm_HandSolder; Mouser Part Number 80-C0603C104J3R -> 81-GCJ188R71H104MA2D; Mouser Price/Stock https://www.mouser.pl/ProductDetail/Murata-Electronics/GRM0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 -> https://www.mouser.pl/pl/ProductDetail/Murata-Electronics/G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
- C40: Mouser Part Number (none) -> 81-GCJ188R71H104MA2D; Mouser Price/Stock https://www.mouser.pl/ProductDetail/Murata-Electronics/GRM0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 -> https://www.mouser.pl/pl/ProductDetail/Murata-Electronics/G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
- C45, C46, C47, C48: Mouser Part Number (none) -> 81-ZRA21CR61E226ME1L; Mouser Price/Stock https://www.mouser.pl/ProductDetail/TDK/C2012X5R1V226M125AC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 -> https://www.mouser.pl/pl/ProductDetail/Murata-Electronics/Z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
