File: hardware/TireTempSensor_v3.0/TireTempSensor_v2.0.kicad_sch (KiCad schematic)
At the start: 19 parts, among them J1 Conn_01x01, J2 Conn_01x01, J3 FTSH-107-01-L-D-K, J4 Conn_01x01, J5 Conn_01x01, U1 STM32G0C1KCTxN, Y1 ATX-11-F-32.000MHZ-F05-T

Commit message: gerber update bo wczesniej nie dzialalo; jeszcze trzeba poprawic tabele z komponentami
Parts:
- C1: footprint Capacitor_SMD:C_0603_1608Metric -> Capacitor_SMD:C_0603_1608Metric_Pad1.08x0.95mm_HandSolder; Mouser Part Number (none) -> 81-ZRB18AR6YA475KE5L; Mouser Price/Stock (none) -> https://www.mouser.pl/pl/ProductDetail/Murata-Electronics/Z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
- C11, C2, C3: footprint Capacitor_SMD:C_0603_1608Metric -> Capacitor_SMD:C_0603_1608Metric_Pad1.08x0.95mm_HandSolder; Mouser Part Number (none) -> 81-GCJ188R71H104MA2D; Mouser Price/Stock (none) -> https://www.mouser.pl/pl/ProductDetail/Murata-Electronics/G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
- C29: value 100nF -> 100n; Mouser Part Number (none) -> 81-GCJ188R71H104MA2D; Mouser Price/Stock (none) -> https://www.mouser.pl/pl/ProductDetail/Murata-Electronics/G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
